File: kicad/EISScube-io.sch (KiCad schematic (older format))
At the start: 7 parts, among them J7 Relay, K1 SANYOU_SRD_Form_C, Q5 GSM3612PJZF

Commit message: Changes for enclosure case
Parts:
- added C27: 104K, Capacitors_SMD:C_0603, symbol C
- added Q4: GSM3612PJZF, TO_SOT_Packages_SMD:SOT-23, symbol Q_NMOS_GSD
- added R18: 100K, Resistors_SMD:R_0603, symbol R
- added R19: 1M, Resistors_SMD:R_0603, symbol R
- added R20: 10K, Resistors_SMD:R_0603, symbol R
Connections:
- net labels added: +1V8, INPUT
- wire segments 24 -> 35
Changed lines of the file:
@@
 $EndDescr
+$Comp
+L GND #PWR013
+U 1 1 5AAC4B4C
+P 2550 3300
+F 0 "#PWR013" H 2550 3050 50  0001 C CNN
+F 1 "GND" H 2550 3150 50  0000 C CNN
+F 2 "" H 2550 3300 50  0001 C CNN
+F 3 "" H 2550 3300 50  0001 C CNN
+	1    2550 3300
+	1    0    0    -1
+$EndComp
 $Comp
 L Q_NMOS_GSD Q5
@@
 	6650 1550 6650 1750
 $Comp
+L Q_NMOS_GSD Q4
+U 1 1 5AAC4B59
+P 2450 2500
+F 0 "Q4" H 2650 2550 50  0000 L CNN
+F 1 "GSM3612PJZF" H 2650 2450 50  0000 L CNN
+F 2 "TO_SOT_Packages_SMD:SOT-23" H 2650 2600 50  0001 C CNN
+F 3 "" H 2450 2500 50  0001 C CNN
+	1    2450 2500
+	1    0    0    -1
+$EndComp
+$Comp
+L R R20
+U 1 1 5AAC62F7
+P 2550 1950
+F 0 "R20" H 2450 1950 50  0000 C CNN
+F 1 "10K" V 2550 1950 50  0000 C CNN
+F 2 "Resistors_SMD:R_0603" V 2480 1950 50  0001 C CNN
+F 3 "" H 2550 1950 50  0001 C CNN
+	1    2550 1950
+	1    0    0    -1
+$EndComp
+$Comp
+L +1V8 #PWR016
+U 1 1 5AAC639B
+P 2550 1650
+F 0 "#PWR016" H 2550 1500 50  0001 C CNN
+F 1 "+1V8" H 2550 1790 50  0000 C CNN
+F 2 "" H 2550 1650 50  0001 C CNN
+F 3 "" H 2550 1650 50  0001 C CNN
+	1    2550 1650
+	1    0    0    -1
+$EndComp
+$Comp
+L R R18
+U 1 1 5AAC4C77
+P 1450 2500
+F 0 "R18" V 1350 2500 50  0000 C CNN
+F 1 "100K" V 1450 2500 50  0000 C CNN
+F 2 "Resistors_SMD:R_0603" V 1380 2500 50  0001 C CNN
+F 3 "" H 1450 2500 50  0001 C CNN
+	1    1450 2500
+	0    1    1    0
+$EndComp
+$Comp
+L R R19
+U 1 1 5AAC4CC1
+P 1800 2850
+F 0 "R19" H 1900 2850 50  0000 C CNN
+F 1 "1M" V 1800 2850 50  0000 C CNN
+F 2 "Resistors_SMD:R_0603" V 1730 2850 50  0001 C CNN
+F 3 "" H 1800 2850 50  0001 C CNN
+	1    1800 2850
+	-1   0    0    1
+$EndComp
+$Comp
+L C C27
+U 1 1 5AAC4D1F
+P 2050 2850
+F 0 "C27" H 1900 2950 50  0000 L CNN
+F 1 "104K" H 2075 2750 50  0000 L CNN
+F 2 "Capacitors_SMD:C_0603" H 2088 2700 50  0001 C CNN
+F 3 "" H 2050 2850 50  0001 C CNN
+	1    2050 2850
+	1    0    0    -1
+$EndComp
+Wire Wire Line
+	2550 1650 2550 1800
+Wire Wire Line
+	2550 2100 2550 2300
+Wire Wire Line
+	1600 2500 2250 2500
+Wire Wire Line
+	1800 2700 1800 2500
+Connection ~ 1800 2500
+Wire Wire Line
+	2050 2700 2050 2500
+Connection ~ 2050 2500
+Wire Wire Line
+	2050 3150 2050 3000
+Wire Wire Line
+	1800 3150 1800 3000
+Wire Wire Line
+	2550 2700 2550 3300
+Connection ~ 2050 3150
+Connection ~ 2550 3150
+Wire Wire Line
+	2550 2200 3150 2200
+Connection ~ 2550 2200
+Text GLabel 3150 2200 2    50   Input ~ 0
+INPUT
+Wire Wire Line
+	1100 2500 1300 2500
+$Comp
 L Conn_01x03 J7
 U 1 1 5AAC5523
@@
 	6300 1650 6650 1650
 Connection ~ 6650 1650
+Wire Wire Line
+	1800 3150 2550 3150
+Text GLabel 1100 2500 0    50   Input ~ 0
+INPUT
 $EndSCHEMATC
