File: kicad/EISScube-cl.sch (KiCad schematic (older format))
At the start: 57 parts, among them J4 SIM_Card_w_det_sw, J5 USB_B_Mini, Q2 GSM3612PJZF, Q3 GSM3612PJZF, Q4 GSM3612PJZF, U3 U-Blox-SARA-R4

Commit message: Changes for enclosure case
Other:
- note added: "Cellular module"
- moved on the sheet: C20, D13, Q4, R13, R14, R15, R18, R19, R25, R27, TP1, TP2

Commit message: changes for new case RL6015
Parts:
- D10, D11, D12, D6, D7, D8, D9: footprint Diodes_SMD:D_0603 -> Inductors_SMD:L_0201
Changed lines of the file:
@@
 F 0 "D6" H 3650 1250 50  0000 L CNN
 F 1 "VBUS05B1-SD0" H 3450 1050 50  0000 L CNN
-F 2 "Diodes_SMD:D_0603" H 3925 1100 50  0001 L CNN
+F 2 "Inductors_SMD:L_0201" H 3925 1100 50  0001 L CNN
 F 3 "" H 3825 1275 50  0001 C CNN
 	1    3700 1150
@@
 F 0 "D7" V 7150 4300 50  0000 L CNN
 F 1 "VBUS05B1-SD0" H 7250 4250 50  0001 L CNN
-F 2 "Diodes_SMD:D_0603" H 7725 4300 50  0001 L CNN
+F 2 "Inductors_SMD:L_0201" H 7725 4300 50  0001 L CNN
 F 3 "" H 7625 4475 50  0001 C CNN
 	1    7500 4350
@@
 F 0 "D8" V 7300 4300 50  0000 L CNN
 F 1 "VBUS05B1-SD0" H 7400 4250 50  0001 L CNN
-F 2 "Diodes_SMD:D_0603" H 7875 4300 50  0001 L CNN
+F 2 "Inductors_SMD:L_0201" H 7875 4300 50  0001 L CNN
 F 3 "" H 7775 4475 50  0001 C CNN
 	1    7650 4350
@@
 F 0 "D9" V 7450 4300 50  0000 L CNN
 F 1 "VBUS05B1-SD0" H 7550 4250 50  0001 L CNN
-F 2 "Diodes_SMD:D_0603" H 8025 4300 50  0001 L CNN
+F 2 "Inductors_SMD:L_0201" H 8025 4300 50  0001 L CNN
 F 3 "" H 7925 4475 50  0001 C CNN
 	1    7800 4350
@@
 F 0 "D10" V 7600 4250 50  0000 L CNN
 F 1 "VBUS05B1-SD0" H 7700 4250 50  0001 L CNN
-F 2 "Diodes_SMD:D_0603" H 8175 4300 50  0001 L CNN
+F 2 "Inductors_SMD:L_0201" H 8175 4300 50  0001 L CNN
 F 3 "" H 8075 4475 50  0001 C CNN
 	1    7950 4350
@@
 F 0 "D11" V 9000 4300 50  0000 L CNN
 F 1 "VBUS05B1-SD0" H 9100 4250 50  0001 L CNN
-F 2 "Diodes_SMD:D_0603" H 9575 4300 50  0001 L CNN
+F 2 "Inductors_SMD:L_0201" H 9575 4300 50  0001 L CNN
 F 3 "" H 9475 4475 50  0001 C CNN
 	1    9350 4350
@@
 F 0 "D12" V 9150 4250 50  0000 L CNN
 F 1 "VBUS05B1-SD0" H 9250 4250 50  0001 L CNN
-F 2 "Diodes_SMD:D_0603" H 9725 4300 50  0001 L CNN
+F 2 "Inductors_SMD:L_0201" H 9725 4300 50  0001 L CNN
 F 3 "" H 9625 4475 50  0001 C CNN
 	1    9500 4350
