File: kicad/EISScube-mc.sch (KiCad schematic (older format))
At the start: 37 parts, among them J1 Boot, J2 UART, J3 JTag, SW1 Reset, U1 STM32L051C8Tx, U2 SN74LV1T34DBVR, U9 LTV-357T, Y1 12MHz, Y2 32.768KHz

Commit message: Changes for enclosure case
Other:
- note added: "Microcontroller"
- moved on the sheet: D18, R2, U9
Changed lines of the file:
@@
 	9950 5900 9950 6100
 Wire Wire Line
-	10100 5800 9950 5800
+	10100 5800 9700 5800
 $Comp
 L C C7
@@
 Text GLabel 2950 4550 0    50   Output ~ 0
 RELAY
-Text GLabel 9950 5800 0    50   UnSpc ~ 0
+Text GLabel 9700 5800 0    50   UnSpc ~ 0
 NRST
 Text GLabel 2750 950  2    50   UnSpc ~ 0
@@
 NoConn ~ 3100 5250
 Wire Wire Line
-	8900 4650 9500 4650
-Wire Wire Line
-	8900 4750 9500 4750
-Wire Wire Line
-	8900 4850 9500 4850
-Wire Wire Line
-	8900 4950 9500 4950
-Text GLabel 9500 4650 2    50   Output ~ 0
+	8900 4650 9450 4650
+Wire Wire Line
+	8900 4750 9450 4750
+Wire Wire Line
+	8900 4850 9450 4850
+Wire Wire Line
+	8900 4950 9450 4950
+Text GLabel 9450 4650 2    50   Output ~ 0
 CL_TXD
-Text GLabel 9500 4750 2    50   Input ~ 0
+Text GLabel 9450 4750 2    50   Input ~ 0
 CL_RXD
-Text GLabel 9500 4850 2    50   Input ~ 0
+Text GLabel 9450 4850 2    50   Input ~ 0
 CL_CTS
-Text GLabel 9500 4950 2    50   Output ~ 0
+Text GLabel 9450 4950 2    50   Output ~ 0
 CL_RTS
 Text Label 9350 5150 2    60   ~ 0
@@
 Wire Wire Line
 	3000 6400 4700 6400
-Text GLabel 7500 900  0    50   Input ~ 0
+Text GLabel 7300 900  0    50   Input ~ 0
 INPUT
 Wire Wire Line
 	9050 3750 8900 3750
-Wire Wire Line
-	8900 900  9150 900
 Wire Wire Line
 	9050 900  9050 3750
@@
 L GND #PWR014
 U 1 1 5ABFAE54
-P 8950 1350
-F 0 "#PWR014" H 8950 1100 50  0001 C CNN
-F 1 "GND" H 8950 1200 50  0000 C CNN
-F 2 "" H 8950 1350 50  0001 C CNN
-F 3 "" H 8950 1350 50  0001 C CNN
-	1    8950 1350
+P 8750 1350
+F 0 "#PWR014" H 8750 1100 50  0001 C CNN
+F 1 "GND" H 8750 1200 50  0000 C CNN
+F 2 "" H 8750 1350 50  0001 C CNN
+F 3 "" H 8750 1350 50  0001 C CNN
+	1    8750 1350
 	1    0    0    -1
 $EndComp
@@
 L GND #PWR015
 U 1 1 5ABFB8ED
-P 8050 1350
-F 0 "#PWR015" H 8050 1100 50  0001 C CNN
-F 1 "GND" H 8050 1200 50  0000 C CNN
-F 2 "" H 8050 1350 50  0001 C CNN
-F 3 "" H 8050 1350 50  0001 C CNN
-	1    8050 1350
+P 7850 1350
+F 0 "#PWR015" H 7850 1100 50  0001 C CNN
+F 1 "GND" H 7850 1200 50  0000 C CNN
+F 2 "" H 7850 1350 50  0001 C CNN
+F 3 "" H 7850 1350 50  0001 C CNN
+	1    7850 1350
 	1    0    0    -1
 $EndComp
@@
 L 1N4001 D18
 U 1 1 5ABFD445
-P 8050 1100
-F 0 "D18" H 8050 1000 50  0000 C CNN
-F 1 "1N4001" H 8050 1200 50  0000 C CNN
-F 2 "Diodes_THT:D_DO-41_SOD81_P10.16mm_Horizontal" H 8050 925 50  0001 C CNN
-F 3 "" H 8050 1100 50  0001 C CNN
-	1    8050 1100
+P 7850 1100
+F 0 "D18" H 7850 1000 50  0000 C CNN
+F 1 "1N4001" H 7850 1200 50  0000 C CNN
+F 2 "Diodes_THT:D_DO-41_SOD81_P10.16mm_Horizontal" H 7850 925 50  0001 C CNN
+F 3 "" H 7850 1100 50  0001 C CNN
+	1    7850 1100
 	0    1    1    0
 $EndComp
@@
 L R R2
 U 1 1 5ABFD67B
-P 7750 900
-F 0 "R2" V 7850 900 50  0000 C CNN
-F 1 "1K" V 7750 900 50  0000 C CNN
-F 2 "Resistors_SMD:R_1206" V 7680 900 50  0001 C CNN
-F 3 "" H 7750 900 50  0001 C CNN
-	1    7750 900
+P 7550 900
+F 0 "R2" V 7650 900 50  0000 C CNN
+F 1 "1K" V 7550 900 50  0000 C CNN
+F 2 "Resistors_SMD:R_1206" V 7480 900 50  0001 C CNN
+F 3 "" H 7550 900 50  0001 C CNN
+	1    7550 900
 	0    -1   -1   0
 $EndComp
 Wire Wire Line
-	7900 900  8300 900
-Wire Wire Line
-	8050 950  8050 900
-Connection ~ 8050 900
-Wire Wire Line
-	8250 1300 8050 1300
-Wire Wire Line
-	8050 1250 8050 1350
-Connection ~ 8050 1300
-Wire Wire Line
-	7600 900  7500 900
+	7700 900  8100 900
+Wire Wire Line
+	7850 950  7850 900
+Connection ~ 7850 900
+Wire Wire Line
+	8050 1300 7850 1300
+Wire Wire Line
+	7850 1250 7850 1350
+Connection ~ 7850 1300
+Wire Wire Line
+	7400 900  7300 900
 $Comp
 L LTV-357T U9
 U 1 1 5ABFA978
-P 8600 1000
-F 0 "U9" H 8550 1200 50  0000 L CNN
-F 1 "LTV-357T" H 8450 800 50  0000 L CNN
-F 2 "Housings_SOIC:SO-4_4.4x3.6mm_Pitch2.54mm" H 8400 800 50  0001 L CIN
-F 3 "" H 8600 1000 50  0001 L CNN
-	1    8600 1000
-	1    0    0    -1
-$EndComp
-Wire Wire Line
-	8900 1100 8950 1100
-Wire Wire Line
-	8950 1100 8950 1350
-Wire Wire Line
-	8300 1100 8250 1100
-Wire Wire Line
-	8250 1100 8250 1300
+P 8400 1000
+F 0 "U9" H 8350 1200 50  0000 L CNN
+F 1 "LTV-357T" H 8250 800 50  0000 L CNN
+F 2 "Housings_SOIC:SO-4_4.4x3.6mm_Pitch2.54mm" H 8200 800 50  0001 L CIN
+F 3 "" H 8400 1000 50  0001 L CNN
+	1    8400 1000
+	1    0    0    -1
+$EndComp
+Wire Wire Line
+	8700 1100 8750 1100
+Wire Wire Line
+	8750 1100 8750 1350
+Wire Wire Line
+	8100 1100 8050 1100
+Wire Wire Line
+	8050 1100 8050 1300
+Wire Wire Line
+	8700 900  9150 900
+Text Notes 5150 750  0    60   ~ 0
+Microcontroller
 $EndSCHEMATC

Commit message: moved LEDs on bottom side. Created a custome bottom part of enclosure RL6015
Connections:
- net +3V3: now also D17.2 (A); no longer R4.2
- net at U1.10 (ADC_IN0/COMP1_INM/COMP1_OUT/RTC_TAMP2/SYS_WKUP1/TIM2_CH1/TIM2_ETR/USART2_CTS/PA0), U9.4: now also R4.1; no longer D17.1 (K)
- new net: D17.1 (K), R4.2
Other:
- moved on the sheet: D17, R4
Changed lines of the file:
@@
 L R R4
 U 1 1 5ABFAF69
-P 9650 900
-F 0 "R4" V 9750 900 50  0000 C CNN
-F 1 "1K" V 9650 900 50  0000 C CNN
-F 2 "Resistors_SMD:R_0603" V 9580 900 50  0001 C CNN
-F 3 "" H 9650 900 50  0001 C CNN
-	1    9650 900
+P 9300 900
+F 0 "R4" V 9400 900 50  0000 C CNN
+F 1 "1K" V 9300 900 50  0000 C CNN
+F 2 "Resistors_SMD:R_0603" V 9230 900 50  0001 C CNN
+F 3 "" H 9300 900 50  0001 C CNN
+	1    9300 900
 	0    -1   -1   0
 $EndComp
@@
 L LED D17
 U 1 1 5ABFBC16
-P 9300 900
-F 0 "D17" H 9300 800 50  0000 C CNN
-F 1 "red" H 9300 800 50  0001 C CNN
-F 2 "LEDs:LED_0603" H 9300 900 50  0001 C CNN
-F 3 "" H 9300 900 50  0001 C CNN
-	1    9300 900
+P 9650 900
+F 0 "D17" H 9650 800 50  0000 C CNN
+F 1 "red" H 9650 800 50  0001 C CNN
+F 2 "LEDs:LED_0603" H 9650 900 50  0001 C CNN
+F 3 "" H 9650 900 50  0001 C CNN
+	1    9650 900
 	1    0    0    1
 $EndComp
-Wire Wire Line
-	9800 900  9850 900
-Wire Wire Line
-	9850 900  9850 850
-Wire Wire Line
-	9500 900  9450 900
 Connection ~ 9050 900
 $Comp
@@
 Text Notes 5150 750  0    60   ~ 0
 Microcontroller
+Wire Wire Line
+	9450 900  9500 900
+Wire Wire Line
+	9800 900  9850 900
+Wire Wire Line
+	9850 900  9850 850
 $EndSCHEMATC
