File: kicad/EISScube-pw.sch (KiCad schematic (older format))
At the start: 33 parts, among them J6 Screw_Terminal_01x08, K1 SANYOU_SRD_Form_C, Q5 GSM3612PJZF, U3 U-Blox-SARA-R4, U4 LM2576HVS-12, U5 MIC29302WU-TR, U6 L7805, U7 LM1117-3.3, U8 LM1117-1.8

Commit message: Changes for enclosure case
Connections:
- net 24VAC-1: now also D14.3 (~~); no longer D14.4 (~~)
- net 24VAC-2: now also D14.4 (~~); no longer D14.3 (~~)
Other:
- note added: "Connector"
- note added: "Power"
- note added: "Relay"
Changed lines of the file:
@@
 	3600 4250 3600 4150
-Wire Wire Line
-	1100 2750 1900 2750
 Wire Wire Line
 	2500 2750 3050 2750
@@
 Wire Wire Line
 	4100 2150 4100 2400
+Text GLabel 1150 1900 0    50   Input ~ 0
+24VAC-1
 Text GLabel 1150 1100 0    50   Input ~ 0
-24VAC-1
-Text GLabel 1150 1900 0    50   Input ~ 0
 24VAC-2
 Text GLabel 4550 1500 2    50   Output ~ 0
@@
 	1    0    0    -1
 $EndComp
-$Comp
-L PWR_FLAG #FLG043
-U 1 1 5AB4CEB6
-P 1100 2750
-F 0 "#FLG043" H 1100 2825 50  0001 C CNN
-F 1 "PWR_FLAG" V 1200 2850 50  0000 C CNN
-F 2 "" H 1100 2750 50  0001 C CNN
-F 3 "" H 1100 2750 50  0001 C CNN
-	1    1100 2750
-	0    -1   -1   0
-$EndComp
 Wire Wire Line
 	7650 1800 9450 1800
@@
 Wire Wire Line
 	3600 6250 3600 5900
+Wire Wire Line
+	1900 2750 1250 2750
+$Comp
+L PWR_FLAG #FLG043
+U 1 1 5AD15A50
+P 3700 1400
+F 0 "#FLG043" H 3700 1475 50  0001 C CNN
+F 1 "PWR_FLAG" H 3700 1550 50  0000 C CNN
+F 2 "" H 3700 1400 50  0001 C CNN
+F 3 "" H 3700 1400 50  0001 C CNN
+	1    3700 1400
+	1    0    0    -1
+$EndComp
+Wire Wire Line
+	3700 1400 3700 1500
+Connection ~ 3700 1500
+Wire Notes Line
+	700  800  5200 800
+Wire Notes Line
+	5200 800  5200 6700
+Wire Notes Line
+	5200 6700 700  6700
+Wire Notes Line
+	700  6700 700  800
+Text Notes 4350 950  0    60   ~ 0
+Power
+Wire Notes Line
+	5400 800  5400 3400
+Wire Notes Line
+	5400 3400 10200 3400
+Wire Notes Line
+	10200 3400 10200 800
+Wire Notes Line
+	10200 800  5400 800
+Text Notes 5700 950  0    60   ~ 0
+Relay
+Text Notes 9400 950  0    60   ~ 0
+Connector
 $EndSCHEMATC

Commit message: changes for new case RL6015
Parts:
- C28: value 470uF 35V -> 220uF 35V
- C30: value 330uF 16V -> 680uF 16V
Changed lines of the file:
@@
 P 2000 1750
 F 0 "C28" H 2025 1850 50  0000 L CNN
-F 1 "470uF 35V" V 2050 1250 50  0000 L CNN
+F 1 "220uF 35V" V 2050 1250 50  0000 L CNN
 F 2 "Capacitors_SMD:CP_Elec_10x10.5" H 2038 1600 50  0001 C CNN
 F 3 "" H 2000 1750 50  0001 C CNN
@@
 P 4100 2000
 F 0 "C30" H 3850 2100 50  0000 L CNN
-F 1 "330uF 16V" V 4250 1750 50  0000 L CNN
+F 1 "680uF 16V" V 4250 1750 50  0000 L CNN
 F 2 "Capacitors_SMD:CP_Elec_10x10.5" H 4138 1850 50  0001 C CNN
 F 3 "" H 4100 2000 50  0001 C CNN

Commit message: moved LEDs on bottom side. Created a custome bottom part of enclosure RL6015
Connections:
- net +12V: now also K1.5
- net at D16.2 (A), R28.1: no longer K1.5
Other:
- moved on the sheet: R28
Changed lines of the file:
@@
 L R R28
 U 1 1 5AB418B7
-P 6750 1300
-F 0 "R28" H 6900 1300 50  0000 C CNN
-F 1 "1K" V 6750 1300 50  0000 C CNN
-F 2 "Resistors_SMD:R_0603" V 6680 1300 50  0001 C CNN
-F 3 "" H 6750 1300 50  0001 C CNN
-	1    6750 1300
+P 6400 1600
+F 0 "R28" H 6550 1600 50  0000 C CNN
+F 1 "1K" V 6400 1600 50  0000 C CNN
+F 2 "Resistors_SMD:R_0603" V 6330 1600 50  0001 C CNN
+F 3 "" H 6400 1600 50  0001 C CNN
+	1    6400 1600
 	-1   0    0    1
 $EndComp
@@
 	7050 1550 7650 1550
 Wire Wire Line
-	6750 1450 6750 1650
-Wire Wire Line
 	7650 1550 7650 1800
 Wire Wire Line
-	6750 1050 6750 1150
-Wire Wire Line
-	6400 1800 6400 1550
-Wire Wire Line
-	6400 1550 6750 1550
-Connection ~ 6750 1550
+	6400 1800 6400 1750
 Wire Wire Line
 	7550 1650 7550 2000
@@
 	3600 6250 3600 5900
 Wire Wire Line
-	1900 2750 1250 2750
+	1250 2750 1900 2750
 $Comp
 L PWR_FLAG #FLG043
@@
 Text Notes 9400 950  0    60   ~ 0
 Connector
+Wire Wire Line
+	6750 1050 6750 1650
+Wire Wire Line
+	6400 1450 6400 1350
+Wire Wire Line
+	6400 1350 6750 1350
+Connection ~ 6750 1350
 $EndSCHEMATC
